File: Class_Projects/Embedded_Systems/DDS_Function_Generator/Discovery_Board_Shield/PCB_Design/2024_Discovery_DDS_Shield/2024_Discovery_DDS_Shield.kicad_pcb (KiCad board)
At the start: 2 copper layers, 98 x 87 mm, 67 parts, among them J1 FILTER_CONN, J2 10118194-0001LF, J3 FTDI_UART_CONN, J4 DC_OFFSET_CONN, J5 LCD_CONN, J6 Conn_OpAmp_Power, J7 Conn_DiscBoard_Right, J8 Conn_DiscBoard_Left, J9 BNC_CONN, SW2 SW_MODE, SW3 SW_CURSOR, SW4 SW_PLUS, SW5 SW_MINUS, SW6 SW_RUN_STOP, U1 TL072, U2 TL072, U5 FT230XS

Commit message: new board version
Parts:
- removed J3: FTDI_UART_CONN, Connector_PinHeader_2.54mm:PinHeader_1x03_P2.54mm_Vertical
- moved C17 11.4 mm to (101.5, 82.1), turned to 0 degrees
- moved R8 2.79 mm to (101.4, 95.6)
- moved R7 2.41 mm to (96.0, 79.9)
- moved C18 2.39 mm to (100.4, 79.8)
- moved D3 2.18 mm to (96.0, 82.2)
- moved D4 1.68 mm to (101.4, 93.3)
Connections:
- D3 pad 1: GND -> Net-(D3-K)
- D4 pad 1: GND -> Net-(D4-K)
- R7 pad 2: Net-(U5-CBUS1) -> /MODE
- R8 pad 2: Net-(U5-CBUS2) -> /MODE
- U5 pad 14: Net-(U5-CBUS1) -> Net-(D3-K)
- U5 pad 7: Net-(U5-CBUS2) -> Net-(D4-K)
Routing:
- net /MODE: track 17.1 -> 42.4 mm, vias 2 -> 4
- net /FTDI_RX: track 35.3 -> 28.1 mm
- net Net-(D4-K): track 0.00 -> 3.59 mm
- net Net-(U5-CBUS2): track 3.15 -> 0.00 mm
- net Net-(D3-K): track 0.00 -> 2.66 mm
- net Net-(U5-CBUS1): track 2.46 -> 0.00 mm
- net /FTDI_TX: track 23.6 -> 21.1 mm
- net GND: track 16.2 -> 14.0 mm, vias 16 -> 14
- net FTDI_VCC: track 24.3 -> 26.0 mm
Other:
- board text added: "May 2024 Embedded Class Version 2.0"
- board text removed: "May 2024 Embedded Class Version 1.0"
- board text removed: "RX"
- board text removed: "TX"
