File: Class_Projects/Embedded_Systems/DDS_Function_Generator/STM32F405_Board/PCB_Design/STM32F405_DDS_Generator/STM32F405_DDS_Generator.kicad_pcb (KiCad board)
At the start: 2 copper layers, 99.1 x 97.1 mm, 121 parts, among them J1 USB_B_Mini, J2 10118194-0001LF, J3 FTDI_UART_CONN, J4 SWD_CONN, J5 LCD_CONN, J6 FILTER_CONN, J7 DC_OFFSET_CONN, J8 BNC_CONN, SW1 SW_RESET, SW2 SW_MODE, SW3 SW_CURSOR, SW4 SW_PLUS, SW5 SW_MINUS, SW6 SW_RUN_STOP, U1 STM32F405RGTx, U2 USBLC6-2SC6, U3 LD1117S33TR_SOT223, U4 TL072, U5 FT230XS, U6 TL072, U7 MC34063AD, Y1 XTAL_8.0MHZ, Y2 XTAL_32.768KHZ

Commit message: updated
Parts:
- removed J3: FTDI_UART_CONN, Connector_PinHeader_2.54mm:PinHeader_1x03_P2.54mm_Vertical
- moved C17 11.3 mm to (114.4, 52.2), turned to 0 degrees
- moved R7 2.82 mm to (108.8, 49.8)
- moved C18 2.74 mm to (113.1, 49.8)
- moved R8 2.34 mm to (114.4, 66.2)
- moved D4 2.18 mm to (114.4, 63.9)
- moved H1 1.97 mm to (122.7, 45.0)
- moved D3 1.83 mm to (108.8, 52.1)
Connections:
- D3 pad 1: GND -> Net-(D3-K)
- D4 pad 1: GND -> Net-(D4-K)
- R7 pad 2: Net-(U5-CBUS1) -> /MODE
- R8 pad 2: Net-(U5-CBUS2) -> /MODE
- U5 pad 14: Net-(U5-CBUS1) -> Net-(D3-K)
- U5 pad 7: Net-(U5-CBUS2) -> Net-(D4-K)
Routing:
- net /MODE: track 17.1 -> 41.7 mm, vias 0 -> 4
- net Net-(D4-K): track 0.00 -> 4.10 mm
- net Net-(U5-CBUS2): track 4.05 -> 0.00 mm, vias 2 -> 0
- net +5V: track 339.2 -> 343.1 mm
- net Net-(D3-K): track 0.00 -> 2.91 mm
- net FTDI_VCC: track 23.6 -> 26.2 mm
- net Net-(U5-CBUS1): track 2.34 -> 0.00 mm
- net GND: track 79.0 -> 76.8 mm, vias 57 -> 55
- net /FTDI_RX: track 42.4 -> 43.1 mm, vias 2 -> 4
- net /FTDI_TX: track 38.2 -> 38.5 mm, vias 4 -> 2
Other:
- board text added: "May 2024 Version 2.0"
- board text removed: "May 2024 Version 1.0"
- board text removed: "RX"
- board text removed: "TX"
