File: Class_Projects/Embedded_Systems/DDS_Function_Generator/STM32F405_Board/PCB_Design/STM32F405_DDS_Generator/STM32F405_DDS_Generator.kicad_sch (KiCad schematic)
At the start: 57 parts, among them J1 USB_B_Mini, J2 10118194-0001LF, J3 FTDI_UART_CONN, J4 SWD_CONN, J5 LCD_CONN, SW1 SW_RESET, SW2 SW_MODE, SW3 SW_CURSOR, SW4 SW_PLUS, SW5 SW_MINUS, SW6 SW_RUN_STOP, U1 STM32F405RGTx, U2 USBLC6-2SC6, U3 LD1117S33TR_SOT223, U5 FT230XS, Y1 XTAL_8.0MHZ, Y2 XTAL_32.768KHZ

Commit message: updated
Parts:
- removed J3: FTDI_UART_CONN, Connector_PinHeader_2.54mm:PinHeader_1x03_P2.54mm_Vertical, symbol Connector_Generic:Conn_01x03
Connections:
- net GND: no longer D3.1 (K), D4.1 (K)
- net MODE: now also R7.2, R8.2
- net at U5.14 (CBUS1): now also D3.1 (K); no longer R7.2
- net at U5.7 (CBUS2): now also D4.1 (K); no longer R8.2
Other:
- moved on the sheet: C17, C18, D3, D4, H1, H2, H3, H4, J2, J4, J5, R10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
