File: Class_Projects/Electronics/2024_NE555_ChargePump/2024_NE555_ChargePump.kicad_pcb (KiCad board)
At the start: 2 copper layers, 87 x 33 mm, 38 parts, among them J1 Vin, J2 Vout, J3 Expansion_Conn, Q1 MMBT2222, U1 NE555D

Commit message: fixes
Parts:
- D1, D10, D11, D12, D3, D4, D5, D6, D7, D8, D9: footprint Diode_SMD:D_MELF -> Diode_SMD:D_MicroMELF_Handsoldering
- Q1: value MMBT2222 -> 2N7002K; footprint MMBT2222:MMBT2222 -> Package_TO_SOT_SMD:SOT-23
- moved Q1 0.13 mm to (125.9, 69.3), turned to 0 degrees
Routing:
- net Net-(D1-K): track 7.87 -> 9.92 mm
- net Net-(D12-K): track 4.03 -> 4.98 mm
- net Net-(D10-A): track 7.24 -> 7.79 mm
- net Net-(D7-K): track 7.06 -> 7.61 mm
