File: Class_Projects/Electronics/2024_NE555_ChargePump/2024_NE555_ChargePump.kicad_sch (KiCad schematic)
At the start: 36 parts, among them J1 Vin, J2 Vout, J3 Expansion_Conn, Q1 MMBT2222, U1 NE555D

Commit message: fixes
Parts:
- removed Q1: MMBT2222, MMBT2222:MMBT2222, symbol MMBT2222:MMBT2222_
- added Q1: 2N7002K, Package_TO_SOT_SMD:SOT-23, symbol Transistor_FET:2N7002K
- D1, D10, D11, D12, D3, D4, D5, D6, D7, D8, D9: footprint Diode_SMD:D_MELF -> Diode_SMD:D_MicroMELF_Handsoldering
Connections:
- net GND: now also Q1.2 (S)
- net SQUARE_1: now also Q1.1 (G)
- net SQUARE_2: now also Q1.3 (D)
Changed lines of the file:
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@@
 	)
 	(junction
-		(at 123.19 45.72)
-		(diameter 0)
-		(color 0 0 0 0)
-	)
-	(junction
 		(at 100.33 101.6)
 		(diameter 0)
@@
 	)
 	(junction
+		(at 123.19 45.72)
+		(diameter 0)
+		(color 0 0 0 0)
+	)
+	(junction
 		(at 58.42 52.07)
 		(diameter 0)
@@
 	(wire
 		(pts
+			(xy 123.19 45.72) (xy 123.19 46.99)
+		)
+		(stroke
+			(width 0)
+			(type default)
+		)
+	)
+	(wire
+		(pts
 			(xy 82.55 101.6) (xy 85.09 101.6)
 		)
@@
 	(wire
 		(pts
+			(xy 123.19 45.72) (xy 135.89 45.72)
+		)
+		(stroke
+			(width 0)
+			(type default)
+		)
+	)
+	(wire
+		(pts
 			(xy 64.77 39.37) (xy 64.77 45.72)
 		)
@@
 	(wire
 		(pts
-			(xy 123.19 45.72) (xy 138.43 45.72)
-		)
-		(stroke
-			(width 0)
-			(type default)
-		)
-	)
-	(wire
-		(pts
 			(xy 27.94 118.11) (xy 49.53 118.11)
 		)
@@
 	(wire
 		(pts
-			(xy 123.19 45.72) (xy 123.19 46.99)
-		)
-		(stroke
-			(width 0)
-			(type default)
-		)
-	)
-	(wire
-		(pts
 			(xy 143.51 36.83) (xy 143.51 38.1)
 		)
@@
 			)
 		)
-		(property "Footprint" "Diode_SMD:D_MELF"
+		(property "Footprint" "Diode_SMD:D_MicroMELF_Handsoldering"
 			(at 88.9 101.6 0)
 			(effects
@@
 			)
 		)
-		(property "Footprint" "Diode_SMD:D_MELF"
+		(property "Footprint" "Diode_SMD:D_MicroMELF_Handsoldering"
 			(at 156.21 101.6 0)
 			(effects
@@
 			)
 		)
-		(property "Footprint" "Diode_SMD:D_MELF"
+		(property "Footprint" "Diode_SMD:D_MicroMELF_Handsoldering"
 			(at 173.99 101.6 0)
 			(effects
@@
 			)
 		)
-		(property "Footprint" "Diode_SMD:D_MELF"
+		(property "Footprint" "Diode_SMD:D_MicroMELF_Handsoldering"
 			(at 55.88 101.6 0)
 			(effects
@@
 			)
 		)
-		(property "Footprint" "Diode_SMD:D_MELF"
+		(property "Footprint" "Diode_SMD:D_MicroMELF_Handsoldering"
 			(at 139.7 101.6 0)
 			(effects
@@
 			)
 		)
-		(property "Footprint" "Diode_SMD:D_MELF"
+		(property "Footprint" "Diode_SMD:D_MicroMELF_Handsoldering"
 			(at 72.39 101.6 0)
 			(effects
@@
 	)
 	(symbol
-		(lib_id "power:GND")
-		(at 97.79 60.96 0)
+		(lib_id "Transistor_FET:2N7002K")
+		(at 140.97 45.72 0)
 		(unit 1)
 		(exclude_from_sim no)
@@
 		(dnp no)
 		(fields_autoplaced yes)
-		(property "Reference" "#PWR06"
-			(at 97.79 67.31 0)
+		(property "Reference" "Q1"
+			(at 147.32 44.4499 0)
 			(effects
 				(font
 					(size 1.27 1.27)
 				)
-				(hide yes)
+				(justify left)
 			)
 		)
-		(property "Value" "GND"
-			(at 97.79 66.04 0)
+		(property "Value" "2N7002K"
+			(at 147.32 46.9899 0)
 			(effects
 				(font
 					(size 1.27 1.27)
 				)
+				(justify left)
 			)
 		)
-		(property "Footprint" ""
-			(at 97.79 60.96 0)
+		(property "Footprint" "Package_TO_SOT_SMD:SOT-23"
+			(at 146.05 47.625 0)
 			(effects
 				(font
 					(size 1.27 1.27)
+					(italic yes)
 				)
+				(justify left)
 				(hide yes)
 			)
 		)
-		(property "Datasheet" ""
-			(at 97.79 60.96 0)
+		(property "Datasheet" "https://www.diodes.com/assets/Datasheets/ds30896.pdf"
+			(at 146.05 49.53 0)
 			(effects
 				(font
 					(size 1.27 1.27)
 				)
+				(justify left)
 				(hide yes)
 			)
 		)
-		(property "Description" "Power symbol creates a global label with name \"GND\" , ground"
-			(at 97.79 60.96 0)
+		(property "Description" "0.38A Id, 60V Vds, N-Channel MOSFET, SOT-23"
+			(at 140.97 45.72 0)
 			(effects
 				(font
@@
 		(pin "1"
 		)
+		(pin "2"
+		)
+		(pin "3"
+		)
 		(instances
 			(project "2024_NE555_ChargePump"
 				(path "/768919b3-6da7-4da6-8803-3d0b98f7ef31"
-					(reference "#PWR06")
+					(reference "Q1")
 					(unit 1)
 				)
@@
 	)
 	(symbol
-		(lib_id "MMBT2222:MMBT2222_")
-		(at 140.97 45.72 0)
+		(lib_id "power:GND")
+		(at 97.79 60.96 0)
 		(unit 1)
 		(exclude_from_sim no)
@@
 		(dnp no)
 		(fields_autoplaced yes)
-		(property "Reference" "Q1"
-			(at 144.78 44.4499 0)
-			(effects
-				(font
-					(size 1.27 1.27)
-				)
-				(justify left)
-			)
-		)
-		(property "Value" "MMBT2222"
-			(at 144.78 46.9899 0)
-			(effects
-				(font
-					(size 1.27 1.27)
-				)
-				(justify left)
-			)
-		)
-		(property "Footprint" "MMBT2222:MMBT2222"
-			(at 140.97 45.72 0)
-			(effects
-				(font
-					(size 1.27 1.27)
-				)
-				(justify bottom)
-				(hide yes)
-			)
-		)
-		(property "Datasheet" ""
-			(at 140.97 45.72 0)
-			(effects
-				(font
-					(size 1.27 1.27)
-				)
-				(hide yes)
-			)
-		)
-		(property "Description" ""
-			(at 140.97 45.72 0)
-			(effects
-				(font
-					(size 1.27 1.27)
-				)
-				(hide yes)
-			)
-		)
-		(property "MF" "ON Semiconductor"
-			(at 140.97 45.72 0)
-			(effects
-				(font
-					(size 1.27 1.27)
-				)
-				(justify bottom)
-				(hide yes)
-			)
-		)
-		(property "Description_1" "\nBipolar (BJT) Transistor NPN 30 V 600 mA 250MHz 300 mW Surface Mount SOT-23-3 (TO-236)\n"
-			(at 140.97 45.72 0)
-			(effects
-				(font
-					(size 1.27 1.27)
-				)
-				(justify bottom)
-				(hide yes)
-			)
-		)
-		(property "Package" "SOT-23-3 Fairchild Semiconductor"
-			(at 140.97 45.72 0)
-			(effects
-				(font
-					(size 1.27 1.27)
-				)
-				(justify bottom)
-				(hide yes)
-			)
-		)
-		(property "Price" "None"
-			(at 140.97 45.72 0)
-			(effects
-				(font
-					(size 1.27 1.27)
-				)
-				(justify bottom)
-				(hide yes)
-			)
-		)
-		(property "SnapEDA_Link" "https://www.snapeda.com/parts/MMBT2222/Onsemi/view-part/?ref=snap"
-			(at 140.97 45.72 0)
+		(property "Reference" "#PWR06"
+			(at 97.79 67.31 0)
 			(effects
 				(font
 					(size 1.27 1.27)
 				)
-				(justify bottom)
 				(hide yes)
 			)
 		)
-		(property "MP" "MMBT2222"
-			(at 140.97 45.72 0)
+		(property "Value" "GND"
+			(at 97.79 66.04 0)
 			(effects
 				(font
 					(size 1.27 1.27)
 				)
-				(justify bottom)
-				(hide yes)
 			)
 		)
-		(property "Purchase-URL" "https://www.snapeda.com/api/url_track_click_mouser/?unipart_id=214298&manufacturer=ON Semiconductor&part_name=MMBT2222&search_term=None"
-			(at 140.97 45.72 0)
+		(property "Footprint" ""
+			(at 97.79 60.96 0)
 			(effects
 				(font
 					(size 1.27 1.27)
 				)
-				(justify bottom)
 				(hide yes)
 			)
 		)
-		(property "Availability" "Not in stock"
-			(at 140.97 45.72 0)
+		(property "Datasheet" ""
+			(at 97.79 60.96 0)
 			(effects
 				(font
 					(size 1.27 1.27)
 				)
-				(justify bottom)
 				(hide yes)
 			)
 		)
-		(property "Check_prices" "https://www.snapeda.com/parts/MMBT2222/Onsemi/view-part/?ref=eda"
-			(at 140.97 45.72 0)
+		(property "Description" "Power symbol creates a global label with name \"GND\" , ground"
+			(at 97.79 60.96 0)
 			(effects
 				(font
 					(size 1.27 1.27)
 				)
-				(justify bottom)
 				(hide yes)
 			)
 		)
-		(pin "B"
-		)
-		(pin "C"
-		)
-		(pin "E"
+		(pin "1"
 		)
 		(instances
 			(project "2024_NE555_ChargePump"
 				(path "/768919b3-6da7-4da6-8803-3d0b98f7ef31"
-					(reference "Q1")
+					(reference "#PWR06")
 					(unit 1)
 				)
@@
 			)
 		)
-		(property "Footprint" "Diode_SMD:D_MELF"
+		(property "Footprint" "Diode_SMD:D_MicroMELF_Handsoldering"
 			(at 33.02 96.52 0)
 			(effects
@@
 			)
 		)
-		(property "Footprint" "Diode_SMD:D_MELF"
+		(property "Footprint" "Diode_SMD:D_MicroMELF_Handsoldering"
 			(at 123.19 101.6 0)
 			(effects
@@
 			)
 		)
-		(property "Footprint" "Diode_SMD:D_MELF"
+		(property "Footprint" "Diode_SMD:D_MicroMELF_Handsoldering"
 			(at 39.37 101.6 0)
 			(effects
@@
 			)
 		)
-		(property "Footprint" "Diode_SMD:D_MELF"
+		(property "Footprint" "Diode_SMD:D_MicroMELF_Handsoldering"
 			(at 190.5 101.6 0)
 			(effects
@@
 			)
 		)
-		(property "Footprint" "Diode_SMD:D_MELF"
+		(property "Footprint" "Diode_SMD:D_MicroMELF_Handsoldering"
 			(at 106.68 101.6 0)
 			(effects
