File: Class_Projects/Electronics/2024_NE555_ChargePump_Expansion/2024_NE555_ChargePump_Expansion.kicad_pcb (KiCad board)
At the start: 2 copper layers, 57 x 35.6 mm, 26 parts, among them J1 Expansion_Conn_In, J2 Vout, J3 Expansion_Conn_Out

Commit message: fixes
Parts:
- D10, D11, D12, D3, D4, D5, D6, D7, D8, D9: footprint Diode_SMD:D_MELF -> Diode_SMD:D_MicroMELF_Handsoldering
Routing:
- net /SQUARE_1: track 68.9 -> 70.7 mm, vias 2 -> 4
- net /Charge_In: track 41.5 -> 42.9 mm
- net Net-(D12-K): track 4.03 -> 4.98 mm
- net Net-(D10-A): track 7.24 -> 7.79 mm
- net Net-(D7-K): track 7.06 -> 7.61 mm
