File: Class_Projects/Electronics/2024_NE555_ChargePump_Expansion/2024_NE555_ChargePump_Expansion.kicad_sch (KiCad schematic)
At the start: 25 parts, among them J1 Expansion_Conn_In, J2 Vout, J3 Expansion_Conn_Out

Commit message: fixes
Parts:
- D10, D11, D12, D3, D4, D5, D6, D7, D8, D9: footprint Diode_SMD:D_MELF -> Diode_SMD:D_MicroMELF_Handsoldering
Changed lines of the file:
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@@
 			)
 		)
-		(property "Footprint" "Diode_SMD:D_MELF"
+		(property "Footprint" "Diode_SMD:D_MicroMELF_Handsoldering"
 			(at 102.87 45.72 0)
 			(effects
@@
 			)
 		)
-		(property "Footprint" "Diode_SMD:D_MELF"
+		(property "Footprint" "Diode_SMD:D_MicroMELF_Handsoldering"
 			(at 170.18 45.72 0)
 			(effects
@@
 			)
 		)
-		(property "Footprint" "Diode_SMD:D_MELF"
+		(property "Footprint" "Diode_SMD:D_MicroMELF_Handsoldering"
 			(at 187.96 45.72 0)
 			(effects
@@
 			)
 		)
-		(property "Footprint" "Diode_SMD:D_MELF"
+		(property "Footprint" "Diode_SMD:D_MicroMELF_Handsoldering"
 			(at 69.85 45.72 0)
 			(effects
@@
 			)
 		)
-		(property "Footprint" "Diode_SMD:D_MELF"
+		(property "Footprint" "Diode_SMD:D_MicroMELF_Handsoldering"
 			(at 153.67 45.72 0)
 			(effects
@@
 			)
 		)
-		(property "Footprint" "Diode_SMD:D_MELF"
+		(property "Footprint" "Diode_SMD:D_MicroMELF_Handsoldering"
 			(at 86.36 45.72 0)
 			(effects
@@
 			)
 		)
-		(property "Footprint" "Diode_SMD:D_MELF"
+		(property "Footprint" "Diode_SMD:D_MicroMELF_Handsoldering"
 			(at 137.16 45.72 0)
 			(effects
@@
 			)
 		)
-		(property "Footprint" "Diode_SMD:D_MELF"
+		(property "Footprint" "Diode_SMD:D_MicroMELF_Handsoldering"
 			(at 53.34 45.72 0)
 			(effects
@@
 			)
 		)
-		(property "Footprint" "Diode_SMD:D_MELF"
+		(property "Footprint" "Diode_SMD:D_MicroMELF_Handsoldering"
 			(at 204.47 45.72 0)
 			(effects
@@
 			)
 		)
-		(property "Footprint" "Diode_SMD:D_MELF"
+		(property "Footprint" "Diode_SMD:D_MicroMELF_Handsoldering"
 			(at 120.65 45.72 0)
 			(effects
