File: Class_Projects/Microprocessors_1/Uno_Shield_DSP_Class_v1/Uno_Shield_DSP_Class_v1.kicad_pcb (KiCad board)
At the start: 2 copper layers, 83.8 x 53.3 mm, 47 parts, among them J1 Power, J10 AudioJack5, J11 AudioJack5, J12 AUDIO_IN, J2 Digital/PWM, J3 Analog, J4 Digital/PWM, J5 IMU_CONN, J6 SCREEN_CONN, J7 AUDIO_OUT, J9 JUMPER, SW1 BT_1, SW2 BT_2, U1 MCP6002-xP

Commit message: gerber
Parts:
- removed R25, R26: 20k, Resistor_THT:R_Axial_DIN0309_L9.0mm_D3.2mm_P2.54mm_Vertical
- R27: value 1k -> 100
Connections:
- RV3 pad 1: Net-(R25-Pad2) -> +5V
- RV3 pad 3: Net-(R26-Pad1) -> GND
Routing:
- net Net-(R25-Pad2): track 15.5 -> 0.00 mm
- net +5V: track 219.1 -> 233.8 mm
- net Net-(R26-Pad1): track 6.85 -> 0.00 mm
