File: Class_Projects/Microprocessors_1/Uno_Shield_DSP_Class_v1/Uno_Shield_DSP_Class_v1.kicad_sch (KiCad schematic)
At the start: 46 parts, among them J1 Power, J10 AudioJack5, J11 AudioJack5, J12 AUDIO_IN, J2 Digital/PWM, J3 Analog, J4 Digital/PWM, J5 IMU_CONN, J6 SCREEN_CONN, J7 AUDIO_OUT, J9 JUMPER, SW1 BT_1, SW2 BT_2, U1 MCP6002-xP

Commit message: gerber
Parts:
- removed R25, R26: 20k, Resistor_THT:R_Axial_DIN0309_L9.0mm_D3.2mm_P2.54mm_Vertical, symbol Device:R_Small
- R27: value 1k -> 100
Connections:
- net +5V: now also RV3.1
- net GND: now also RV3.3
Changed lines of the file:
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@@
 	(wire
 		(pts
-			(xy 137.16 149.86) (xy 137.16 151.13)
-		)
-		(stroke
-			(width 0)
-			(type default)
-		)
-	)
-	(wire
-		(pts
 			(xy 77.47 111.76) (xy 77.47 113.03)
 		)
@@
 	(wire
 		(pts
-			(xy 137.16 128.27) (xy 137.16 129.54)
-		)
-		(stroke
-			(width 0)
-			(type default)
-		)
-	)
-	(wire
-		(pts
 			(xy 85.09 113.03) (xy 86.36 113.03)
 		)
@@
 	(wire
 		(pts
-			(xy 137.16 134.62) (xy 137.16 135.89)
+			(xy 137.16 133.35) (xy 137.16 135.89)
 		)
 		(stroke
@@
 			)
 		)
-		(property "Value" "1k"
+		(property "Value" "100"
 			(at 178.054 119.634 90)
 			(effects
@@
 	(symbol
 		(lib_id "power:+5V")
-		(at 137.16 128.27 0)
+		(at 137.16 133.35 0)
 		(unit 1)
 		(exclude_from_sim no)
@@
 		(dnp no)
 		(property "Reference" "#PWR026"
-			(at 137.16 132.08 0)
+			(at 137.16 137.16 0)
 			(effects
 				(font
@@
 		)
 		(property "Value" "+5V"
-			(at 137.5156 125.222 90)
+			(at 137.5156 130.302 90)
 			(effects
 				(font
@@
 		)
 		(property "Footprint" ""
-			(at 137.16 128.27 0)
+			(at 137.16 133.35 0)
 			(effects
 				(font
@@
 		)
 		(property "Datasheet" ""
-			(at 137.16 128.27 0)
+			(at 137.16 133.35 0)
 			(effects
 				(font
@@
 		)
 		(property "Description" "Power symbol creates a global label with name \"+5V\""
-			(at 137.16 128.27 0)
+			(at 137.16 133.35 0)
 			(effects
 				(font
@@
 	)
 	(symbol
-		(lib_id "Device:R_Small")
-		(at 137.16 132.08 0)
-		(unit 1)
-		(exclude_from_sim no)
-		(in_bom yes)
-		(on_board yes)
-		(dnp no)
-		(property "Reference" "R25"
-			(at 134.112 130.81 0)
-			(effects
-				(font
-					(size 1.016 1.016)
-				)
-			)
-		)
-		(property "Value" "20k"
-			(at 133.858 132.842 0)
-			(effects
-				(font
-					(size 1.27 1.27)
-				)
-			)
-		)
-		(property "Footprint" "Resistor_THT:R_Axial_DIN0309_L9.0mm_D3.2mm_P2.54mm_Vertical"
-			(at 137.16 132.08 0)
-			(effects
-				(font
-					(size 1.27 1.27)
-				)
-				(hide yes)
-			)
-		)
-		(property "Datasheet" "~"
-			(at 137.16 132.08 0)
-			(effects
-				(font
-					(size 1.27 1.27)
-				)
-				(hide yes)
-			)
-		)
-		(property "Description" "Resistor, small symbol"
-			(at 137.16 132.08 0)
-			(effects
-				(font
-					(size 1.27 1.27)
-				)
-				(hide yes)
-			)
-		)
-		(pin "2"
-		)
-		(pin "1"
-		)
-		(instances
-			(project "Uno_Shield_DSP_Class_v1"
-				(path "/e63e39d7-6ac0-4ffd-8aa3-1841a4541b55"
-					(reference "R25")
-					(unit 1)
-				)
-			)
-		)
-	)
-	(symbol
 		(lib_name "AudioJack5_1")
 		(lib_id "Connector_Audio:AudioJack5")
@@
 	(symbol
 		(lib_id "power:GND")
-		(at 137.16 151.13 0)
+		(at 137.16 144.78 0)
 		(unit 1)
 		(exclude_from_sim no)
@@
 		(dnp no)
 		(property "Reference" "#PWR025"
-			(at 137.16 157.48 0)
+			(at 137.16 151.13 0)
 			(effects
 				(font
@@
 		)
 		(property "Value" "GND"
-			(at 137.16 155.194 0)
+			(at 137.16 148.844 0)
 			(effects
 				(font
@@
 		)
 		(property "Footprint" ""
-			(at 137.16 151.13 0)
+			(at 137.16 144.78 0)
 			(effects
 				(font
@@
 		)
 		(property "Datasheet" ""
-			(at 137.16 151.13 0)
+			(at 137.16 144.78 0)
 			(effects
 				(font
@@
 		)
 		(property "Description" "Power symbol creates a global label with name \"GND\" , ground"
-			(at 137.16 151.13 0)
+			(at 137.16 144.78 0)
 			(effects
 				(font
@@
 					(unit 1)
 				)
-			)
-		)
-	)
-	(symbol
-		(lib_id "Device:R_Small")
-		(at 137.16 147.32 0)
-		(unit 1)
-		(exclude_from_sim no)
-		(in_bom yes)
-		(on_board yes)
-		(dnp no)
-		(property "Reference" "R26"
-			(at 134.112 146.05 0)
-			(effects
-				(font
-					(size 1.016 1.016)
-				)
-			)
-		)
-		(property "Value" "20k"
-			(at 133.858 148.082 0)
-			(effects
-				(font
-					(size 1.27 1.27)
-				)
-			)
-		)
-		(property "Footprint" "Resistor_THT:R_Axial_DIN0309_L9.0mm_D3.2mm_P2.54mm_Vertical"
-			(at 137.16 147.32 0)
-			(effects
-				(font
-					(size 1.27 1.27)
-				)
-				(hide yes)
-			)
-		)
-		(property "Datasheet" "~"
-			(at 137.16 147.32 0)
-			(effects
-				(font
-					(size 1.27 1.27)
-				)
-				(hide yes)
-			)
-		)
-		(property "Description" "Resistor, small symbol"
-			(at 137.16 147.32 0)
-			(effects
-				(font
-					(size 1.27 1.27)
-				)
-				(hide yes)
-			)
-		)
-		(pin "2"
-		)
-		(pin "1"
-		)
-		(instances
-			(project "Uno_Shield_DSP_Class_v1"
-				(path "/e63e39d7-6ac0-4ffd-8aa3-1841a4541b55"
-					(reference "R26")
-					(unit 1)
-				)
